Commit message: 🍱 updatae assets

File: src/silverscreen/assets/gr1/urdf/fourier_left_hand.urdf (robot description, URDF)
Before this commit: robot fourier_hand_left, 17 links, 16 joints
Links:
- link L_index_intermediate: mass 0.012927 -> 0.012925; geometry collision mesh filename=../meshes/fourier_hand/L_index_intermediate.STL; visual mesh filename=../meshes/fourier_hand/L_index_intermediate.STL
- link L_index_proximal: mass 0.019118 -> 0.019117; geometry collision mesh filename=../meshes/fourier_hand/L_index_proximal.STL; visual mesh filename=../meshes/fourier_hand/L_index_proximal.STL
- link L_middle_intermediate: geometry collision mesh filename=../meshes/fourier_hand/L_middle_intermediate.STL; visual mesh filename=../meshes/fourier_hand/L_middle_intermediate.STL
- link L_middle_proximal: geometry collision mesh filename=../meshes/fourier_hand/L_middle_proximal.STL; visual mesh filename=../meshes/fourier_hand/L_middle_proximal.STL
- link L_pinky_intermediate: mass 0.0056868 -> 0.0056869; geometry collision mesh filename=../meshes/fourier_hand/L_pinky_intermediate.STL; visual mesh filename=../meshes/fourier_hand/L_pinky_intermediate.STL
- link L_pinky_proximal: geometry collision mesh filename=../meshes/fourier_hand/L_pinky_proximal.STL; visual mesh filename=../meshes/fourier_hand/L_pinky_proximal.STL
- link L_ring_intermediate: mass 0.012926 -> 0.012927; geometry collision mesh filename=../meshes/fourier_hand/L_ring_intermediate.STL; visual mesh filename=../meshes/fourier_hand/L_ring_intermediate.STL
- link L_ring_proximal: mass 0.019117 -> 0.019118; geometry collision mesh filename=../meshes/fourier_hand/L_ring_proximal.STL; visual mesh filename=../meshes/fourier_hand/L_ring_proximal.STL
- link L_thumb_distal: geometry collision mesh filename=../meshes/fourier_hand/L_thumb_distal.STL; visual mesh filename=../meshes/fourier_hand/L_thumb_distal.STL
- link L_thumb_proximal: geometry collision mesh filename=../meshes/fourier_hand/L_thumb_proximal.STL; visual mesh filename=../meshes/fourier_hand/L_thumb_proximal.STL
- link L_thumb_proximal_base: geometry collision mesh filename=../meshes/fourier_hand/L_thumb_proximal_base.STL; visual mesh filename=../meshes/fourier_hand/L_thumb_proximal_base.STL
- link l_hand_base_link: mass 0.099947 -> 0.09995; geometry collision mesh filename=../meshes/fourier_hand/l_hand_base_link.STL; visual mesh filename=../meshes/fourier_hand/l_hand_base_link.STL
Joints:
- joint L_index_intermediate_joint: origin xyz=0.0315316061985493 -0.00545507200132231 0 rpy=0 0 -6.82553680074393E-05 -> xyz=0.031532 -0.0054551 0 rpy=0 0 -6.8255E-05
- joint L_index_proximal_joint: origin xyz=0.026869067504082 -0.0122934392405636 -0.0959894118552304 rpy=0.00130566300740641 1.51842419415245 0.00130387280614764 -> xyz=0.026869 -0.012293 -0.095989 rpy=0.0013057 1.5184 0.0013039
- joint L_index_tip_joint: origin xyz=0.038 -0.0038 0 rpy=0 0 0 -> xyz=0.038 -0.001 0 rpy=0 0 0
- joint L_middle_intermediate_joint: origin xyz=0.0316616941629316 -0.00464081056852417 0 rpy=0 0 -6.83490817261459E-05 -> xyz=0.031662 -0.0046408 0 rpy=0 0 -6.8349E-05
- joint L_middle_proximal_joint: origin xyz=0.00850119653118567 -0.0122933023251572 -0.0979925903933238 rpy=1.39401189702948 1.57072689557984 1.3940118966122 -> xyz=0.0085012 -0.012293 -0.097993 rpy=1.394 1.5707 1.394
- joint L_middle_tip_joint: origin xyz=0.045 -0.0032 0 rpy=0 0 0 -> xyz=0.045 0.0005 0 rpy=0 0 0
- joint L_pinky_intermediate_joint: origin xyz=0.0313378020543266 -0.00647627689369765 0 rpy=0 0 -6.79747455421694E-05 -> xyz=0.031338 -0.0064763 0 rpy=0 0 -6.7975E-05
- joint L_pinky_proximal_joint: origin xyz=-0.0282266675554703 -0.012293437629494 -0.0960129830601813 rpy=3.14093869761107 1.46608875997235 3.14094227921624 -> xyz=-0.028227 -0.012293 -0.096013 rpy=3.1409 1.4661 3.1409
- joint L_pinky_tip_joint: origin xyz=0.031 -0.007 0 rpy=0 0 0 -> xyz=0.031 -0.0045 0 rpy=0 0 0
- joint L_ring_intermediate_joint: origin xyz=0.0315316061985493 -0.00545507200132236 0 rpy=0 0 -6.82554553643455E-05 -> xyz=0.031532 -0.0054551 0 rpy=0 0 -6.8255E-05
- joint L_ring_proximal_joint: origin xyz=-0.0099599699075906 -0.012293306060256 -0.0979379429013024 rpy=3.14028638202668 1.51844861517835 3.14028817139281 -> xyz=-0.00996 -0.012293 -0.097938 rpy=3.1403 1.5184 3.1403
- joint L_ring_tip_joint: origin xyz=0.038 -0.0038 0 rpy=0 0 0 -> xyz=0.038 -0.002 0 rpy=0 0 0
- joint L_thumb_distal_joint: origin xyz=0.0615493701717829 0.00746157030770586 0 rpy=0 0 1.22106056547031E-05 -> xyz=0.061549 0.0074616 0 rpy=0 0 1.221E-05
- joint L_thumb_proximal_pitch_joint: origin xyz=0.02175 0 0 rpy=-1.57072797771317 0 0 -> xyz=0.02175 0 0 rpy=-1.5707 0 0
- joint L_thumb_proximal_yaw_joint: origin xyz=0.0220003063830263 -0.0154982849769962 -0.0250926444440346 rpy=0 -1.22105233317497E-05 0 -> xyz=0.022 -0.015498 -0.025093 rpy=0 -1.2211E-05 0

File: src/silverscreen/assets/gr1/urdf/fourier_right_hand.urdf (robot description, URDF)
Before this commit: robot fourier_hand_right, 17 links, 16 joints
Links:
- link R_index_intermediate: geometry collision mesh filename=../meshes/fourier_hand/R_index_intermediate.STL; visual mesh filename=../meshes/fourier_hand/R_index_intermediate.STL
- link R_index_proximal: geometry collision mesh filename=../meshes/fourier_hand/R_index_proximal.STL; visual mesh filename=../meshes/fourier_hand/R_index_proximal.STL
- link R_middle_intermediate: geometry collision mesh filename=../meshes/fourier_hand/R_middle_intermediate.STL; visual mesh filename=../meshes/fourier_hand/R_middle_intermediate.STL
- link R_middle_proximal: geometry collision mesh filename=../meshes/fourier_hand/R_middle_proximal.STL; visual mesh filename=../meshes/fourier_hand/R_middle_proximal.STL
- link R_pinky_intermediate: geometry collision mesh filename=../meshes/fourier_hand/R_pinky_intermediate.STL; visual mesh filename=../meshes/fourier_hand/R_pinky_intermediate.STL
- link R_pinky_proximal: geometry collision mesh filename=../meshes/fourier_hand/R_pinky_proximal.STL; visual mesh filename=../meshes/fourier_hand/R_pinky_proximal.STL
- link R_ring_intermediate: geometry collision mesh filename=../meshes/fourier_hand/R_ring_intermediate.STL; visual mesh filename=../meshes/fourier_hand/R_ring_intermediate.STL
- link R_ring_proximal: geometry collision mesh filename=../meshes/fourier_hand/R_ring_proximal.STL; visual mesh filename=../meshes/fourier_hand/R_ring_proximal.STL
- link R_thumb_distal: geometry collision mesh filename=../meshes/fourier_hand/R_thumb_distal.STL; visual mesh filename=../meshes/fourier_hand/R_thumb_distal.STL
- link R_thumb_proximal: geometry collision mesh filename=../meshes/fourier_hand/R_thumb_proximal.STL; visual mesh filename=../meshes/fourier_hand/R_thumb_proximal.STL
- link R_thumb_proximal_base: geometry collision mesh filename=../meshes/fourier_hand/R_thumb_proximal_base.STL; visual mesh filename=../meshes/fourier_hand/R_thumb_proximal_base.STL
- link r_hand_base_link: geometry collision mesh filename=../meshes/fourier_hand/r_hand_base_link.STL; visual mesh filename=../meshes/fourier_hand/r_hand_base_link.STL
Joints:
- joint R_index_intermediate_joint: origin xyz=0.0315316061985493 -0.00545507200132231 0 rpy=0 0 0 -> xyz=0.031532 -0.0054551 0 rpy=0 0 0
- joint R_index_proximal_joint: axis 0.0012744819545806 0.219189646097979 0.975681441219003 -> 0 0 1; origin xyz=0.0268347443648602 0.01238126080166 -0.0959877257832576 rpy=-3.14028763091841 1.5184240046093 0.00408527869771669 -> xyz=0.026583 0.012307 -0.096064 rpy=-3.1402 1.5214 0.0013813
- joint R_index_tip_joint: origin xyz=0.038 -0.0038 0 rpy=0 0 0 -> xyz=0.038 -0.0015 0 rpy=0 0 0
- joint R_middle_intermediate_joint: origin xyz=0.0316616941629307 -0.00464081056853635 0 rpy=0 0 0 -> xyz=0.031662 -0.0046408 0 rpy=0 0 0
- joint R_middle_proximal_joint: origin xyz=0.00846694447258024 0.0123302974668429 -0.0979909078036594 rpy=-1.75035301585144 1.57072689472437 1.39402168267738 -> xyz=0.0082089 0.012307 -0.098014 rpy=-0.023406 1.5679 3.1182
- joint R_middle_tip_joint: origin xyz=0.045 -0.0032 0 rpy=0 0 0 -> xyz=0.045 0.0005 0 rpy=0 0 0
- joint R_pinky_intermediate_joint: origin xyz=0.0314990327566104 -0.00564011838510353 0 rpy=0 0 0.0263892434774018 -> xyz=0.031338 -0.0064763 0 rpy=0 0 6.7954E-05
- joint R_pinky_proximal_joint: origin xyz=-0.0282607774805067 0.012227983776169 -0.0960113074336258 rpy=-0.248599525552003 1.46275517858851 2.89438415643823 -> xyz=-0.028513 0.012307 -0.095926 rpy=-0.00063622 1.4632 3.141
- joint R_pinky_tip_joint: origin xyz=0.031 -0.007 0 rpy=0 0 0 -> xyz=0.031 -0.004 0 rpy=0 0 0
- joint R_ring_intermediate_joint: origin xyz=0.0315320280251494 -0.00545263318234326 0 rpy=0 0 0 -> xyz=0.031531 -0.0054572 0 rpy=0 0 0
- joint R_ring_proximal_joint: origin xyz=-0.00999415052356634 0.0122789339975533 -0.0979362638116289 rpy=-0.00278180898871791 1.51844864673705 3.14159265358979 -> xyz=-0.010252 0.012307 -0.097905 rpy=0 1.5155 3.1416
- joint R_ring_tip_joint: origin xyz=0.038 -0.0038 0 rpy=0 0 0 -> xyz=0.038 -0.0015 0 rpy=0 0 0
- joint R_thumb_distal_joint: origin xyz=0.0614443264755605 0.00828219439307844 0 rpy=0 0 1.22100084212751E-05 -> xyz=0.061444 0.0082822 0 rpy=0 0 -0.0029196
- joint R_thumb_proximal_pitch_joint: origin xyz=0.0217499931849152 -1.72158354079244E-05 0 rpy=1.57086466715046 1.22641020904056E-05 -0.000791532745143911 -> xyz=0.02175 -1.722E-05 6.35E-05 rpy=1.5709 -0.0029195 -0.00079174
- joint R_thumb_proximal_yaw_joint: axis -1.22100045962969E-05 6.83500415353481E-05 0.999999997589594 -> 0 0 1; origin xyz=0.0219570995851234 0.0155628599102215 -0.0250905219673082 rpy=3.14159265358979 0 0 -> xyz=0.021922 0.015502 -0.025153 rpy=3.1416 0 0

File: src/silverscreen/assets/gr1/urdf/robot.urdf (robot description, URDF)
Before this commit: robot GR1T2_fourier_hand_capsule_coll, 71 links, 70 joints
Links:
- link L_index_intermediate: mass 0.012927 -> 0.012925; geometry collision mesh filename=../meshes/fourier_hand/L_index_intermediate.STL; visual mesh filename=../meshes/fourier_hand/L_index_intermediate.STL
- link L_index_proximal: mass 0.019118 -> 0.019117; geometry collision mesh filename=../meshes/fourier_hand/L_index_proximal.STL; visual mesh filename=../meshes/fourier_hand/L_index_proximal.STL
- link L_middle_intermediate: geometry collision mesh filename=../meshes/fourier_hand/L_middle_intermediate.STL; visual mesh filename=../meshes/fourier_hand/L_middle_intermediate.STL
- link L_middle_proximal: geometry collision mesh filename=../meshes/fourier_hand/L_middle_proximal.STL; visual mesh filename=../meshes/fourier_hand/L_middle_proximal.STL
- link L_pinky_intermediate: mass 0.0056868 -> 0.0056869; geometry collision mesh filename=../meshes/fourier_hand/L_pinky_intermediate.STL; visual mesh filename=../meshes/fourier_hand/L_pinky_intermediate.STL
- link L_pinky_proximal: geometry collision mesh filename=../meshes/fourier_hand/L_pinky_proximal.STL; visual mesh filename=../meshes/fourier_hand/L_pinky_proximal.STL
- link L_ring_intermediate: mass 0.012926 -> 0.012927; geometry collision mesh filename=../meshes/fourier_hand/L_ring_intermediate.STL; visual mesh filename=../meshes/fourier_hand/L_ring_intermediate.STL
- link L_ring_proximal: mass 0.019117 -> 0.019118; geometry collision mesh filename=../meshes/fourier_hand/L_ring_proximal.STL; visual mesh filename=../meshes/fourier_hand/L_ring_proximal.STL
- link L_thumb_distal: geometry collision mesh filename=../meshes/fourier_hand/L_thumb_distal.STL; visual mesh filename=../meshes/fourier_hand/L_thumb_distal.STL
- link L_thumb_proximal: geometry collision mesh filename=../meshes/fourier_hand/L_thumb_proximal.STL; visual mesh filename=../meshes/fourier_hand/L_thumb_proximal.STL
- link L_thumb_proximal_base: geometry collision mesh filename=../meshes/fourier_hand/L_thumb_proximal_base.STL; visual mesh filename=../meshes/fourier_hand/L_thumb_proximal_base.STL
- link R_index_intermediate: geometry collision mesh filename=../meshes/fourier_hand/R_index_intermediate.STL; visual mesh filename=../meshes/fourier_hand/R_index_intermediate.STL
- link R_index_proximal: geometry collision mesh filename=../meshes/fourier_hand/R_index_proximal.STL; visual mesh filename=../meshes/fourier_hand/R_index_proximal.STL
- link R_middle_intermediate: geometry collision mesh filename=../meshes/fourier_hand/R_middle_intermediate.STL; visual mesh filename=../meshes/fourier_hand/R_middle_intermediate.STL
- link R_middle_proximal: geometry collision mesh filename=../meshes/fourier_hand/R_middle_proximal.STL; visual mesh filename=../meshes/fourier_hand/R_middle_proximal.STL
- link R_pinky_intermediate: geometry collision mesh filename=../meshes/fourier_hand/R_pinky_intermediate.STL; visual mesh filename=../meshes/fourier_hand/R_pinky_intermediate.STL
- link R_pinky_proximal: geometry collision mesh filename=../meshes/fourier_hand/R_pinky_proximal.STL; visual mesh filename=../meshes/fourier_hand/R_pinky_proximal.STL
- link R_ring_intermediate: geometry collision mesh filename=../meshes/fourier_hand/R_ring_intermediate.STL; visual mesh filename=../meshes/fourier_hand/R_ring_intermediate.STL
- link R_ring_proximal: geometry collision mesh filename=../meshes/fourier_hand/R_ring_proximal.STL; visual mesh filename=../meshes/fourier_hand/R_ring_proximal.STL
- link R_thumb_distal: geometry collision mesh filename=../meshes/fourier_hand/R_thumb_distal.STL; visual mesh filename=../meshes/fourier_hand/R_thumb_distal.STL
- link R_thumb_proximal: geometry collision mesh filename=../meshes/fourier_hand/R_thumb_proximal.STL; visual mesh filename=../meshes/fourier_hand/R_thumb_proximal.STL
- link R_thumb_proximal_base: geometry collision mesh filename=../meshes/fourier_hand/R_thumb_proximal_base.STL; visual mesh filename=../meshes/fourier_hand/R_thumb_proximal_base.STL
- link base_link: mass 4.72 -> 3.96
- link l_hand_base_link: mass 0.099947 -> 0.09995; geometry collision mesh filename=../meshes/fourier_hand/l_hand_base_link.STL; visual mesh filename=../meshes/fourier_hand/l_hand_base_link.STL
- link left_hand_yaw_link: mass 0.86 -> 0.99
- link left_shank_pitch_link: mass 2.35 -> 1.76
- link left_thigh_pitch_link: mass 9.66 -> 8.35; geometry collision cylinder length=0.24982894507630515 radius=0.082; visual mesh filename=../meshes/left_thigh_pitch_link.STL
- link left_thigh_roll_link: mass 1.86 -> 1.47
- link left_thigh_yaw_link: mass 1.85 -> 3.47
- link r_hand_base_link: geometry collision mesh filename=../meshes/fourier_hand/r_hand_base_link.STL; visual mesh filename=../meshes/fourier_hand/r_hand_base_link.STL
- link right_hand_yaw_link: mass 0.86 -> 0.99
- link right_shank_pitch_link: mass 2.35 -> 1.76
- link right_thigh_pitch_link: mass 9.66 -> 8.35; geometry collision cylinder length=0.24982123520352716 radius=0.082; visual mesh filename=../meshes/right_thigh_pitch_link.STL
- link right_thigh_roll_link: mass 1.86 -> 1.47
- link right_thigh_yaw_link: mass 1.85 -> 3.47
- link torso_link: mass 5.118 -> 5.67
Joints:
- joint L_index_intermediate_joint: origin xyz=0.0315316061985493 -0.00545507200132231 0 rpy=0 0 -6.82553680074393E-05 -> xyz=0.031532 -0.0054551 0 rpy=0 0 -6.8255E-05
- joint L_index_proximal_joint: origin xyz=0.026869067504082 -0.0122934392405636 -0.0959894118552304 rpy=0.00130566300740641 1.51842419415245 0.00130387280614764 -> xyz=0.026869 -0.012293 -0.095989 rpy=0.0013057 1.5184 0.0013039
- joint L_index_tip_joint: origin xyz=0.038 -0.0038 0 rpy=0 0 0 -> xyz=0.038 -0.001 0 rpy=0 0 0
- joint L_middle_intermediate_joint: origin xyz=0.0316616941629316 -0.00464081056852417 0 rpy=0 0 -6.83490817261459E-05 -> xyz=0.031662 -0.0046408 0 rpy=0 0 -6.8349E-05
- joint L_middle_proximal_joint: origin xyz=0.00850119653118567 -0.0122933023251572 -0.0979925903933238 rpy=1.39401189702948 1.57072689557984 1.3940118966122 -> xyz=0.0085012 -0.012293 -0.097993 rpy=1.394 1.5707 1.394
- joint L_middle_tip_joint: origin xyz=0.045 -0.0032 0 rpy=0 0 0 -> xyz=0.045 0.0005 0 rpy=0 0 0
- joint L_pinky_intermediate_joint: origin xyz=0.0313378020543266 -0.00647627689369765 0 rpy=0 0 -6.79747455421694E-05 -> xyz=0.031338 -0.0064763 0 rpy=0 0 -6.7975E-05
- joint L_pinky_proximal_joint: origin xyz=-0.0282266675554703 -0.012293437629494 -0.0960129830601813 rpy=3.14093869761107 1.46608875997235 3.14094227921624 -> xyz=-0.028227 -0.012293 -0.096013 rpy=3.1409 1.4661 3.1409
- joint L_pinky_tip_joint: origin xyz=0.031 -0.007 0 rpy=0 0 0 -> xyz=0.031 -0.0045 0 rpy=0 0 0
- joint L_ring_intermediate_joint: origin xyz=0.0315316061985493 -0.00545507200132236 0 rpy=0 0 -6.82554553643455E-05 -> xyz=0.031532 -0.0054551 0 rpy=0 0 -6.8255E-05
- joint L_ring_proximal_joint: origin xyz=-0.0099599699075906 -0.012293306060256 -0.0979379429013024 rpy=3.14028638202668 1.51844861517835 3.14028817139281 -> xyz=-0.00996 -0.012293 -0.097938 rpy=3.1403 1.5184 3.1403
- joint L_ring_tip_joint: origin xyz=0.038 -0.0038 0 rpy=0 0 0 -> xyz=0.038 -0.002 0 rpy=0 0 0
- joint L_thumb_distal_joint: origin xyz=0.0615493701717829 0.00746157030770586 0 rpy=0 0 1.22106056547031E-05 -> xyz=0.061549 0.0074616 0 rpy=0 0 1.221E-05
- joint L_thumb_proximal_pitch_joint: origin xyz=0.02175 0 0 rpy=-1.57072797771317 0 0 -> xyz=0.02175 0 0 rpy=-1.5707 0 0
- joint L_thumb_proximal_yaw_joint: origin xyz=0.0220003063830263 -0.0154982849769962 -0.0250926444440346 rpy=0 -1.22105233317497E-05 0 -> xyz=0.022 -0.015498 -0.025093 rpy=0 -1.2211E-05 0
- joint R_index_intermediate_joint: origin xyz=0.0315316061985493 -0.00545507200132231 0 rpy=0 0 0 -> xyz=0.031532 -0.0054551 0 rpy=0 0 0
- joint R_index_proximal_joint: axis 0.0012744819545806 0.219189646097979 0.975681441219003 -> 0 0 1; origin xyz=0.0268347443648602 0.01238126080166 -0.0959877257832576 rpy=-3.14028763091841 1.5184240046093 0.00408527869771669 -> xyz=0.026583 0.012307 -0.096064 rpy=-3.1402 1.5214 0.0013813
- joint R_index_tip_joint: origin xyz=0.038 -0.0038 0 rpy=0 0 0 -> xyz=0.038 -0.0015 0 rpy=0 0 0
- joint R_middle_intermediate_joint: origin xyz=0.0316616941629307 -0.00464081056853635 0 rpy=0 0 0 -> xyz=0.031662 -0.0046408 0 rpy=0 0 0
- joint R_middle_proximal_joint: origin xyz=0.00846694447258024 0.0123302974668429 -0.0979909078036594 rpy=-1.75035301585144 1.57072689472437 1.39402168267738 -> xyz=0.0082089 0.012307 -0.098014 rpy=-0.023406 1.5679 3.1182
- joint R_middle_tip_joint: origin xyz=0.045 -0.0032 0 rpy=0 0 0 -> xyz=0.045 0.0005 0 rpy=0 0 0
- joint R_pinky_intermediate_joint: origin xyz=0.0314990327566104 -0.00564011838510353 0 rpy=0 0 0.0263892434774018 -> xyz=0.031338 -0.0064763 0 rpy=0 0 6.7954E-05
- joint R_pinky_proximal_joint: origin xyz=-0.0282607774805067 0.012227983776169 -0.0960113074336258 rpy=-0.248599525552003 1.46275517858851 2.89438415643823 -> xyz=-0.028513 0.012307 -0.095926 rpy=-0.00063622 1.4632 3.141
- joint R_pinky_tip_joint: origin xyz=0.031 -0.007 0 rpy=0 0 0 -> xyz=0.031 -0.004 0 rpy=0 0 0
- joint R_ring_intermediate_joint: origin xyz=0.0315320280251494 -0.00545263318234326 0 rpy=0 0 0 -> xyz=0.031531 -0.0054572 0 rpy=0 0 0
- joint R_ring_proximal_joint: origin xyz=-0.00999415052356634 0.0122789339975533 -0.0979362638116289 rpy=-0.00278180898871791 1.51844864673705 3.14159265358979 -> xyz=-0.010252 0.012307 -0.097905 rpy=0 1.5155 3.1416
- joint R_ring_tip_joint: origin xyz=0.038 -0.0038 0 rpy=0 0 0 -> xyz=0.038 -0.0015 0 rpy=0 0 0
- joint R_thumb_distal_joint: origin xyz=0.0614443264755605 0.00828219439307844 0 rpy=0 0 1.22100084212751E-05 -> xyz=0.061444 0.0082822 0 rpy=0 0 -0.0029196
- joint R_thumb_proximal_pitch_joint: origin xyz=0.0217499931849152 -1.72158354079244E-05 0 rpy=1.57086466715046 1.22641020904056E-05 -0.000791532745143911 -> xyz=0.02175 -1.722E-05 6.35E-05 rpy=1.5709 -0.0029195 -0.00079174
- joint R_thumb_proximal_yaw_joint: axis -1.22100045962969E-05 6.83500415353481E-05 0.999999997589594 -> 0 0 1; origin xyz=0.0219570995851234 0.0155628599102215 -0.0250905219673082 rpy=3.14159265358979 0 0 -> xyz=0.021922 0.015502 -0.025153 rpy=3.1416 0 0
- joint imu_joint: origin xyz=0 0 -0.0596 rpy=0 0 0 -> xyz=0 0 -0.0595999999999995 rpy=0 0 0
- joint l_hand_base_joint: origin xyz=-0.00143750472419189 -5.94019892983799E-05 -0.0210000216633744 rpy=0 0 0 -> xyz=-0.0014375 -5.9402E-05 -0.021 rpy=0 0 0
- joint left_ankle_pitch_joint: origin xyz=3.2116E-05 -0.00125 -0.34 rpy=0 0 0 -> xyz=0 -0.00125 -0.34 rpy=0 0 0
- joint left_elbow_pitch_joint: origin xyz=0 0.0051 -0.1786 rpy=0 0 0 -> xyz=0 0.0010503 -0.1786 rpy=0 0 0
- joint left_hip_pitch_joint: origin xyz=0 0.0408 -0.14027 rpy=0 0 0 -> xyz=0 0.0223 -0.14027 rpy=0 0 0
- joint left_hip_yaw_joint: origin xyz=0.033135 -7.7152E-05 0.00075 rpy=0 0 0 -> xyz=0.033135 0 0.00075 rpy=0 0 0
- joint left_knee_pitch_joint: origin xyz=0 -0.039262 -0.36 rpy=0 0 0 -> xyz=0 -0.019512 -0.36 rpy=0 0 0
- joint left_shoulder_roll_joint: limit lower=-0.57 upper=2.53 effort=38 velocity=9.11 -> lower=-0.57 upper=3.27 effort=38 velocity=9.11; origin xyz=0.00085 0.09515 0 rpy=-0.43275 0 0 -> xyz=0 0.09515 0 rpy=-0.43275 0 0
- joint left_shoulder_yaw_joint: origin xyz=-0.00085 0.04 -0.0749 rpy=0 0 0 -> xyz=0 0.04 -0.0709 rpy=0 0 0
- joint left_wrist_yaw_joint: origin xyz=0 -0.0040497 -0.05945 rpy=0 0 0 -> xyz=0 0 -0.05945 rpy=0 0 0
- joint r_hand_base_joint: origin xyz=-0.00141711624232485 0 -0.0210000172555634 rpy=0 0 0 -> xyz=-0.0014094 0 -0.021 rpy=-6.835E-05 -0.0029196 0
- joint right_elbow_pitch_joint: origin xyz=0 -0.0051 -0.1786 rpy=0 0 0 -> xyz=0 -0.0010503 -0.1786 rpy=0 0 0
- joint right_hip_pitch_joint: origin xyz=0 -0.0408 -0.14027 rpy=0 0 0 -> xyz=0 -0.0223 -0.14027 rpy=0 0 0
- joint right_knee_pitch_joint: origin xyz=0 0.039512 -0.36 rpy=0 0 0 -> xyz=0 0.019762 -0.36 rpy=0 0 0
- joint right_shoulder_pitch_joint: origin xyz=0 -0.10094 0.047376 rpy=-0.43992 0 0 -> xyz=0 -0.10128 0.046651 rpy=-0.43275 0 0
- joint right_shoulder_roll_joint: limit lower=-2.53 upper=0.57 effort=38 velocity=9.11 -> lower=-3.27 upper=0.57 effort=38 velocity=9.11; origin xyz=0.00085 -0.09515 0 rpy=0.43992 0 0 -> xyz=0 -0.09515 0 rpy=0.43275 0 0
- joint right_shoulder_yaw_joint: origin xyz=-0.00085 -0.04 -0.0709 rpy=0 0 0 -> xyz=0 -0.04 -0.0709 rpy=0 0 0
- joint right_wrist_roll_joint: origin xyz=0 0 -0.19021 rpy=0 0 0 -> xyz=0 0 -0.19115 rpy=0 0 0
- joint right_wrist_yaw_joint: origin xyz=0 0.0040497 -0.05945 rpy=0 0 0 -> xyz=0 0 -0.05945 rpy=0 0 0
- joint waist_pitch_joint: origin xyz=0 0.00335 0.0927 rpy=0 0 0 -> xyz=0 0 0.0869 rpy=0 0 0
- joint waist_roll_joint: origin xyz=0.00525 -0.00385 0.0752 rpy=0 0 0 -> xyz=0.00525 -0.0005 0.081 rpy=0 0 0
