Commit message: 🍱 update urdfs and inspire hand urdf
Signed-off-by: Yuxiang Gao <yuxiang.gao@fftai.com>

File: assets/gr1/urdf/GR1T2_fourier_hand_6dof.urdf (robot description, URDF)
Before this commit: robot GR1T2_fourier_hand, 71 links, 70 joints
Links:
- removed link L_index_intermediate
- removed link L_index_proximal
- removed link L_index_tip
- removed link L_middle_intermediate
- removed link L_middle_proximal
- removed link L_middle_tip
- removed link L_pinky_intermediate
- removed link L_pinky_proximal
- removed link L_pinky_tip
- removed link L_ring_intermediate
- removed link L_ring_proximal
- removed link L_ring_tip
- removed link L_thumb_distal
- removed link L_thumb_proximal
- removed link L_thumb_proximal_base
- removed link L_thumb_tip
- removed link R_index_intermediate
- removed link R_index_proximal
- removed link R_index_tip
- removed link R_middle_intermediate
- removed link R_middle_proximal
- removed link R_middle_tip
- removed link R_pinky_intermediate
- removed link R_pinky_proximal
- removed link R_pinky_tip
- removed link R_ring_intermediate
- removed link R_ring_proximal
- removed link R_ring_tip
- removed link R_thumb_distal
- removed link R_thumb_proximal
- removed link R_thumb_proximal_base
- removed link R_thumb_tip
- removed link l_hand_base_link
- removed link r_hand_base_link
- added link L_hand_base_link, mass 0.306; collision mesh filename=../meshes/fourier_hand_6dof/L_hand_base_link.STL; visual mesh filename=../meshes/fourier_hand_6dof/L_hand_base_link.STL
- added link L_index_intermediate_link, mass 0.01292544; collision mesh filename=../meshes/fourier_hand_6dof/L_index_intermediate_link.STL; visual mesh filename=../meshes/fourier_hand_6dof/L_index_intermediate_link.STL
- added link L_index_proximal_link, mass 0.019117; collision mesh filename=../meshes/fourier_hand_6dof/L_index_proximal_link.STL; visual mesh filename=../meshes/fourier_hand_6dof/L_index_proximal_link.STL
- added link L_index_tip_link; visual sphere radius=0.005
- added link L_middle_intermediate_link, mass 0.01535007; collision mesh filename=../meshes/fourier_hand_6dof/L_middle_intermediate_link.STL; visual mesh filename=../meshes/fourier_hand_6dof/L_middle_intermediate_link.STL
- added link L_middle_proximal_link, mass 0.01911771; collision mesh filename=../meshes/fourier_hand_6dof/L_middle_proximal_link.STL; visual mesh filename=../meshes/fourier_hand_6dof/L_middle_proximal_link.STL
- added link L_middle_tip_link; visual sphere radius=0.005
- added link L_pinky_intermediate_link, mass 0.00568707; collision mesh filename=../meshes/fourier_hand_6dof/L_pinky_intermediate_link.STL; visual mesh filename=../meshes/fourier_hand_6dof/L_pinky_intermediate_link.STL
- added link L_pinky_proximal_link, mass 0.01911771; collision mesh filename=../meshes/fourier_hand_6dof/L_pinky_proximal_link.STL; visual mesh filename=../meshes/fourier_hand_6dof/L_pinky_proximal_link.STL
- added link L_pinky_tip_link; visual sphere radius=0.005
- added link L_ring_intermediate_link, mass 0.01292544; collision mesh filename=../meshes/fourier_hand_6dof/L_ring_intermediate_link.STL; visual mesh filename=../meshes/fourier_hand_6dof/L_ring_intermediate_link.STL
- added link L_ring_proximal_link, mass 0.01911771; collision mesh filename=../meshes/fourier_hand_6dof/L_ring_proximal_link.STL; visual mesh filename=../meshes/fourier_hand_6dof/L_ring_proximal_link.STL
- added link L_ring_tip_link; visual sphere radius=0.005
- added link L_thumb_distal_link, mass 0.02031766; collision mesh filename=../meshes/fourier_hand_6dof/L_thumb_distal_link.STL; visual mesh filename=../meshes/fourier_hand_6dof/L_thumb_distal_link.STL
- added link L_thumb_proximal_base_link, mass 0.00948527; collision mesh filename=../meshes/fourier_hand_6dof/L_thumb_proximal_base_link.STL; visual mesh filename=../meshes/fourier_hand_6dof/L_thumb_proximal_base_link.STL
- added link L_thumb_proximal_link, mass 0.07347612; collision mesh filename=../meshes/fourier_hand_6dof/L_thumb_proximal_link.STL; visual mesh filename=../meshes/fourier_hand_6dof/L_thumb_proximal_link.STL
- added link L_thumb_tip_link; visual sphere radius=0.005
- added link R_hand_base_link, mass 0.306; collision mesh filename=../meshes/fourier_hand_6dof/R_hand_base_link.STL; visual mesh filename=../meshes/fourier_hand_6dof/R_hand_base_link.STL
- added link R_index_intermediate_link, mass 0.01292544; collision mesh filename=../meshes/fourier_hand_6dof/R_index_intermediate_link.STL; visual mesh filename=../meshes/fourier_hand_6dof/R_index_intermediate_link.STL
- added link R_index_proximal_link, mass 0.01911771; collision mesh filename=../meshes/fourier_hand_6dof/R_index_proximal_link.STL; visual mesh filename=../meshes/fourier_hand_6dof/R_index_proximal_link.STL
- added link R_index_tip_link; visual sphere radius=0.005
- added link R_middle_intermediate_link, mass 0.01535; collision mesh filename=../meshes/fourier_hand_6dof/R_middle_intermediate_link.STL; visual mesh filename=../meshes/fourier_hand_6dof/R_middle_intermediate_link.STL
- added link R_middle_proximal_link, mass 0.01911771; collision mesh filename=../meshes/fourier_hand_6dof/R_middle_proximal_link.STL; visual mesh filename=../meshes/fourier_hand_6dof/R_middle_proximal_link.STL
- added link R_middle_tip_link; visual sphere radius=0.005
- added link R_pinky_intermediate_link, mass 0.00568707; collision mesh filename=../meshes/fourier_hand_6dof/R_pinky_intermediate_link.STL; visual mesh filename=../meshes/fourier_hand_6dof/R_pinky_intermediate_link.STL
- added link R_pinky_proximal_link, mass 0.01911771; collision mesh filename=../meshes/fourier_hand_6dof/R_pinky_proximal_link.STL; visual mesh filename=../meshes/fourier_hand_6dof/R_pinky_proximal_link.STL
- added link R_pinky_tip_link; visual sphere radius=0.005
- added link R_ring_intermediate_link, mass 0.012925; collision mesh filename=../meshes/fourier_hand_6dof/R_ring_intermediate_link.STL; visual mesh filename=../meshes/fourier_hand_6dof/R_ring_intermediate_link.STL
- added link R_ring_proximal_link, mass 0.01911771; collision mesh filename=../meshes/fourier_hand_6dof/R_ring_proximal_link.STL; visual mesh filename=../meshes/fourier_hand_6dof/R_ring_proximal_link.STL
- added link R_ring_tip_link; visual sphere radius=0.005
- added link R_thumb_distal_link, mass 0.01974135; collision mesh filename=../meshes/fourier_hand_6dof/R_thumb_distal_link.STL; visual mesh filename=../meshes/fourier_hand_6dof/R_thumb_distal_link.STL
- added link R_thumb_proximal_base_link, mass 0.00948218; collision mesh filename=../meshes/fourier_hand_6dof/R_thumb_proximal_base_link.STL; visual mesh filename=../meshes/fourier_hand_6dof/R_thumb_proximal_base_link.STL
- added link R_thumb_proximal_link, mass 0.07405243; collision mesh filename=../meshes/fourier_hand_6dof/R_thumb_proximal_link.STL; visual mesh filename=../meshes/fourier_hand_6dof/R_thumb_proximal_link.STL
- added link R_thumb_tip_link; visual sphere radius=0.005
Joints:
- removed joint l_hand_base_joint
- removed joint r_hand_base_joint
- added joint L_hand_base_joint: type fixed, parent left_end_effector_link, child L_hand_base_link, origin xyz=0 0 -0.021 rpy=0 0 0, axis 0 0 0
- added joint R_hand_base_joint: type fixed, parent right_end_effector_link, child R_hand_base_link, origin xyz=0 0 -0.0210000000049082 rpy=-6.83500415935726E-05 1.22100046026127E-05 0, axis 0 0 0
- joint L_index_intermediate_joint: child L_index_intermediate -> L_index_intermediate_link; origin xyz=0.031532 -0.0054551 0 rpy=0 0 -6.8255E-05 -> xyz=0.031532 -0.0054551 0 rpy=0 0 -6.8256E-05; parent L_index_proximal -> L_index_proximal_link
- joint L_index_proximal_joint: child L_index_proximal -> L_index_proximal_link; parent l_hand_base_link -> L_hand_base_link
- joint L_index_tip_joint: child L_index_tip -> L_index_tip_link; origin xyz=0.038 -0.001 0 rpy=0 0 0 -> xyz=0.038 -0.0015 0 rpy=0 0 0; parent L_index_intermediate -> L_index_intermediate_link
- joint L_middle_intermediate_joint: child L_middle_intermediate -> L_middle_intermediate_link; origin xyz=0.031662 -0.0046408 0 rpy=0 0 -6.8349E-05 -> xyz=0.031662 -0.0046408 0 rpy=0 0 -6.835E-05; parent L_middle_proximal -> L_middle_proximal_link
- joint L_middle_proximal_joint: child L_middle_proximal -> L_middle_proximal_link; parent l_hand_base_link -> L_hand_base_link
- joint L_middle_tip_joint: child L_middle_tip -> L_middle_tip_link; parent L_middle_intermediate -> L_middle_intermediate_link
- joint L_pinky_intermediate_joint: child L_pinky_intermediate -> L_pinky_intermediate_link; origin xyz=0.031338 -0.0064763 0 rpy=0 0 -6.7975E-05 -> xyz=0.031338 -0.0064763 0 rpy=0 0 -6.7976E-05; parent L_pinky_proximal -> L_pinky_proximal_link
- joint L_pinky_proximal_joint: child L_pinky_proximal -> L_pinky_proximal_link; parent l_hand_base_link -> L_hand_base_link
- joint L_pinky_tip_joint: child L_pinky_tip -> L_pinky_tip_link; origin xyz=0.031 -0.0045 0 rpy=0 0 0 -> xyz=0.031 -0.0040 0 rpy=0 0 0; parent L_pinky_intermediate -> L_pinky_intermediate_link
- joint L_ring_intermediate_joint: child L_ring_intermediate -> L_ring_intermediate_link; origin xyz=0.031532 -0.0054551 0 rpy=0 0 -6.8255E-05 -> xyz=0.031532 -0.0054551 0 rpy=0 0 -6.8256E-05; parent L_ring_proximal -> L_ring_proximal_link
- joint L_ring_proximal_joint: child L_ring_proximal -> L_ring_proximal_link; parent l_hand_base_link -> L_hand_base_link
- joint L_ring_tip_joint: child L_ring_tip -> L_ring_tip_link; parent L_ring_intermediate -> L_ring_intermediate_link
- joint L_thumb_distal_joint: child L_thumb_distal -> L_thumb_distal_link; limit lower=0 upper=1.04 effort=10 velocity=0.8 -> lower=0 upper=1.23 effort=10 velocity=0.8; parent L_thumb_proximal -> L_thumb_proximal_link
- joint L_thumb_proximal_pitch_joint: child L_thumb_proximal -> L_thumb_proximal_link; parent L_thumb_proximal_base -> L_thumb_proximal_base_link
- joint L_thumb_proximal_yaw_joint: child L_thumb_proximal_base -> L_thumb_proximal_base_link; origin xyz=0.022 -0.015498 -0.025093 rpy=0 -1.2211E-05 0 -> xyz=0.022 -0.015498 -0.025093 rpy=0 -1.221E-05 0; parent l_hand_base_link -> L_hand_base_link
- joint L_thumb_tip_joint: child L_thumb_tip -> L_thumb_tip_link; origin xyz=0.031 0 0 rpy=0 0 0 -> xyz=0.031 -0.001 0 rpy=0 0 0; parent L_thumb_distal -> L_thumb_distal_link
- joint R_index_intermediate_joint: child R_index_intermediate -> R_index_intermediate_link; parent R_index_proximal -> R_index_proximal_link
- joint R_index_proximal_joint: child R_index_proximal -> R_index_proximal_link; origin xyz=0.026583 0.012307 -0.096064 rpy=-3.1402 1.5214 0.0013813 -> xyz=0.026864 0.012307 -0.095892 rpy=-3.1403 1.5184 0.0013039; parent r_hand_base_link -> R_hand_base_link
- joint R_index_tip_joint: child R_index_tip -> R_index_tip_link; parent R_index_intermediate -> R_index_intermediate_link
- joint R_middle_intermediate_joint: child R_middle_intermediate -> R_middle_intermediate_link; parent R_middle_proximal -> R_middle_proximal_link
- joint R_middle_proximal_joint: child R_middle_proximal -> R_middle_proximal_link; origin xyz=0.0082089 0.012307 -0.098014 rpy=-0.023406 1.5679 3.1182 -> xyz=0.0084962 0.012307 -0.097896 rpy=-1.7476 1.5707 1.394; parent r_hand_base_link -> R_hand_base_link
- joint R_middle_tip_joint: child R_middle_tip -> R_middle_tip_link; parent R_middle_intermediate -> R_middle_intermediate_link
- joint R_pinky_intermediate_joint: child R_pinky_intermediate -> R_pinky_intermediate_link; origin xyz=0.031338 -0.0064763 0 rpy=0 0 6.7954E-05 -> xyz=0.031338 -0.0064763 0 rpy=0 0 6.7976E-05; parent R_pinky_proximal -> R_pinky_proximal_link
- joint R_pinky_proximal_joint: child R_pinky_proximal -> R_pinky_proximal_link; origin xyz=-0.028513 0.012307 -0.095926 rpy=-0.00063622 1.4632 3.141 -> xyz=-0.028232 0.012307 -0.095916 rpy=-0.00065397 1.4661 3.1409; parent r_hand_base_link -> R_hand_base_link
- joint R_pinky_tip_joint: child R_pinky_tip -> R_pinky_tip_link; parent R_pinky_intermediate -> R_pinky_intermediate_link
- joint R_ring_intermediate_joint: child R_ring_intermediate -> R_ring_intermediate_link; parent R_ring_proximal -> R_ring_proximal_link
- joint R_ring_proximal_joint: child R_ring_proximal -> R_ring_proximal_link; origin xyz=-0.010252 0.012307 -0.097905 rpy=0 1.5155 3.1416 -> xyz=-0.009965 0.012307 -0.097841 rpy=0 1.5184 3.1416; parent r_hand_base_link -> R_hand_base_link
- joint R_ring_tip_joint: child R_ring_tip -> R_ring_tip_link; parent R_ring_intermediate -> R_ring_intermediate_link
- joint R_thumb_distal_joint: child R_thumb_distal -> R_thumb_distal_link; limit lower=0 upper=1.04 effort=10 velocity=0.8 -> lower=0 upper=1.23 effort=10 velocity=0.8; origin xyz=0.061444 0.0082822 0 rpy=0 0 -0.0029196 -> xyz=0.061444 0.0082822 0 rpy=0 0 1.221E-05; parent R_thumb_proximal -> R_thumb_proximal_link
- joint R_thumb_proximal_pitch_joint: child R_thumb_proximal -> R_thumb_proximal_link; origin xyz=0.02175 -1.722E-05 6.35E-05 rpy=1.5709 -0.0029195 -0.00079174 -> xyz=0.02175 0 0 rpy=1.5709 1.221E-05 0; parent R_thumb_proximal_base -> R_thumb_proximal_base_link
- joint R_thumb_proximal_yaw_joint: child R_thumb_proximal_base -> R_thumb_proximal_base_link; origin xyz=0.021922 0.015502 -0.025153 rpy=3.1416 0 0 -> xyz=0.021995 0.015502 -0.024995 rpy=3.1416 0 0; parent r_hand_base_link -> R_hand_base_link
- joint R_thumb_tip_joint: child R_thumb_tip -> R_thumb_tip_link; parent R_thumb_distal -> R_thumb_distal_link
- joint left_shoulder_roll_joint: limit lower=-0.57 upper=3.27 effort=38 velocity=9.11 -> lower=-0.57 upper=2.53 effort=38 velocity=9.11
- joint left_wrist_pitch_joint: limit lower=-0.96 upper=0.87 effort=3.95 velocity=27.96 -> lower=-0.61 upper=0.61 effort=3.95 velocity=27.96
- joint left_wrist_roll_joint: limit lower=-0.61 upper=0.61 effort=3.95 velocity=27.96 -> lower=-0.87 upper=0.96 effort=3.95 velocity=27.96
- joint right_shoulder_roll_joint: limit lower=-3.27 upper=0.57 effort=38 velocity=9.11 -> lower=-2.53 upper=0.57 effort=38 velocity=9.11
- joint right_wrist_pitch_joint: limit lower=-0.96 upper=0.87 effort=3.95 velocity=27.96 -> lower=-0.61 upper=0.61 effort=3.95 velocity=27.96
- joint right_wrist_roll_joint: limit lower=-0.61 upper=0.61 effort=3.95 velocity=27.96 -> lower=-0.96 upper=0.87 effort=3.95 velocity=27.96

File: assets/gr1/urdf/fourier_left_hand_6dof.urdf (robot description, URDF)
Before this commit: robot fourier_right_hand, 17 links, 16 joints
Links:
- removed link R_index_intermediate
- removed link R_index_proximal
- removed link R_index_tip
- removed link R_middle_intermediate
- removed link R_middle_proximal
- removed link R_middle_tip
- removed link R_pinky_intermediate
- removed link R_pinky_proximal
- removed link R_pinky_tip
- removed link R_ring_intermediate
- removed link R_ring_proximal
- removed link R_ring_tip
- removed link R_thumb_distal
- removed link R_thumb_proximal
- removed link R_thumb_proximal_base
- removed link R_thumb_tip
- removed link r_hand_base_link
- added link L_hand_base_link, mass 0.306; collision mesh filename=../meshes/fourier_hand_6dof/L_hand_base_link.STL; visual mesh filename=../meshes/fourier_hand_6dof/L_hand_base_link.STL
- added link L_index_intermediate_link, mass 0.01292544; collision mesh filename=../meshes/fourier_hand_6dof/L_index_intermediate_link.STL; visual mesh filename=../meshes/fourier_hand_6dof/L_index_intermediate_link.STL
- added link L_index_proximal_link, mass 0.019117; collision mesh filename=../meshes/fourier_hand_6dof/L_index_proximal_link.STL; visual mesh filename=../meshes/fourier_hand_6dof/L_index_proximal_link.STL
- added link L_index_tip_link; visual sphere radius=0.005
- added link L_middle_intermediate_link, mass 0.01535007; collision mesh filename=../meshes/fourier_hand_6dof/L_middle_intermediate_link.STL; visual mesh filename=../meshes/fourier_hand_6dof/L_middle_intermediate_link.STL
- added link L_middle_proximal_link, mass 0.01911771; collision mesh filename=../meshes/fourier_hand_6dof/L_middle_proximal_link.STL; visual mesh filename=../meshes/fourier_hand_6dof/L_middle_proximal_link.STL
- added link L_middle_tip_link; visual sphere radius=0.005
- added link L_pinky_intermediate_link, mass 0.00568707; collision mesh filename=../meshes/fourier_hand_6dof/L_pinky_intermediate_link.STL; visual mesh filename=../meshes/fourier_hand_6dof/L_pinky_intermediate_link.STL
- added link L_pinky_proximal_link, mass 0.01911771; collision mesh filename=../meshes/fourier_hand_6dof/L_pinky_proximal_link.STL; visual mesh filename=../meshes/fourier_hand_6dof/L_pinky_proximal_link.STL
- added link L_pinky_tip_link; visual sphere radius=0.005
- added link L_ring_intermediate_link, mass 0.01292544; collision mesh filename=../meshes/fourier_hand_6dof/L_ring_intermediate_link.STL; visual mesh filename=../meshes/fourier_hand_6dof/L_ring_intermediate_link.STL
- added link L_ring_proximal_link, mass 0.01911771; collision mesh filename=../meshes/fourier_hand_6dof/L_ring_proximal_link.STL; visual mesh filename=../meshes/fourier_hand_6dof/L_ring_proximal_link.STL
- added link L_ring_tip_link; visual sphere radius=0.005
- added link L_thumb_distal_link, mass 0.02031766; collision mesh filename=../meshes/fourier_hand_6dof/L_thumb_distal_link.STL; visual mesh filename=../meshes/fourier_hand_6dof/L_thumb_distal_link.STL
- added link L_thumb_proximal_base_link, mass 0.00948527; collision mesh filename=../meshes/fourier_hand_6dof/L_thumb_proximal_base_link.STL; visual mesh filename=../meshes/fourier_hand_6dof/L_thumb_proximal_base_link.STL
- added link L_thumb_proximal_link, mass 0.07347612; collision mesh filename=../meshes/fourier_hand_6dof/L_thumb_proximal_link.STL; visual mesh filename=../meshes/fourier_hand_6dof/L_thumb_proximal_link.STL
- added link L_thumb_tip_link; visual sphere radius=0.005
Joints:
- removed joint R_index_intermediate_joint
- removed joint R_index_proximal_joint
- removed joint R_index_tip_joint
- removed joint R_middle_intermediate_joint
- removed joint R_middle_proximal_joint
- removed joint R_middle_tip_joint
- removed joint R_pinky_intermediate_joint
- removed joint R_pinky_proximal_joint
- removed joint R_pinky_tip_joint
- removed joint R_ring_intermediate_joint
- removed joint R_ring_proximal_joint
- removed joint R_ring_tip_joint
- removed joint R_thumb_distal_joint
- removed joint R_thumb_proximal_pitch_joint
- removed joint R_thumb_proximal_yaw_joint
- removed joint R_thumb_tip_joint
- added joint L_index_intermediate_joint: type revolute, parent L_index_proximal_link, child L_index_intermediate_link, origin xyz=0.031532 -0.0054551 0 rpy=0 0 -6.8256E-05, axis 0 0 1, limit lower=-1.74 upper=0 effort=10 velocity=0.8, mimic joint=L_index_proximal_joint multiplier=1.128 offset=0
- added joint L_index_proximal_joint: type revolute, parent L_hand_base_link, child L_index_proximal_link, origin xyz=0.026869 -0.012293 -0.095989 rpy=0.0013057 1.5184 0.0013039, axis 0 0 1, limit lower=-1.57 upper=0 effort=10 velocity=0.8
- added joint L_index_tip_joint: type fixed, parent L_index_intermediate_link, child L_index_tip_link, origin xyz=0.038 -0.0015 0 rpy=0 0 0
- added joint L_middle_intermediate_joint: type revolute, parent L_middle_proximal_link, child L_middle_intermediate_link, origin xyz=0.031662 -0.0046408 0 rpy=0 0 -6.835E-05, axis 0 0 1, limit lower=-1.74 upper=0 effort=10 velocity=0.8, mimic joint=L_middle_proximal_joint multiplier=1.131 offset=0
- added joint L_middle_proximal_joint: type revolute, parent L_hand_base_link, child L_middle_proximal_link, origin xyz=0.0085012 -0.012293 -0.097993 rpy=1.394 1.5707 1.394, axis 0 0 1, limit lower=-1.57 upper=0 effort=10 velocity=0.8
- added joint L_middle_tip_joint: type fixed, parent L_middle_intermediate_link, child L_middle_tip_link, origin xyz=0.045 0.0005 0 rpy=0 0 0
- added joint L_pinky_intermediate_joint: type revolute, parent L_pinky_proximal_link, child L_pinky_intermediate_link, origin xyz=0.031338 -0.0064763 0 rpy=0 0 -6.7976E-05, axis 0 0 1, limit lower=-1.74 upper=0 effort=10 velocity=0.8, mimic joint=L_pinky_proximal_joint multiplier=1.129 offset=0
- added joint L_pinky_proximal_joint: type revolute, parent L_hand_base_link, child L_pinky_proximal_link, origin xyz=-0.028227 -0.012293 -0.096013 rpy=3.1409 1.4661 3.1409, axis 0 0 1, limit lower=-1.57 upper=0 effort=10 velocity=0.8
- added joint L_pinky_tip_joint: type fixed, parent L_pinky_intermediate_link, child L_pinky_tip_link, origin xyz=0.031 -0.0040 0 rpy=0 0 0
- added joint L_ring_intermediate_joint: type revolute, parent L_ring_proximal_link, child L_ring_intermediate_link, origin xyz=0.031532 -0.0054551 0 rpy=0 0 -6.8256E-05, axis 0 0 1, limit lower=-1.74 upper=0 effort=10 velocity=0.8, mimic joint=L_ring_proximal_joint multiplier=1.143 offset=0
- added joint L_ring_proximal_joint: type revolute, parent L_hand_base_link, child L_ring_proximal_link, origin xyz=-0.00996 -0.012293 -0.097938 rpy=3.1403 1.5184 3.1403, axis 0 0 1, limit lower=-1.57 upper=0 effort=10 velocity=0.8
- added joint L_ring_tip_joint: type fixed, parent L_ring_intermediate_link, child L_ring_tip_link, origin xyz=0.038 -0.002 0 rpy=0 0 0
- added joint L_thumb_distal_joint: type revolute, parent L_thumb_proximal_link, child L_thumb_distal_link, origin xyz=0.061549 0.0074616 0 rpy=0 0 1.221E-05, axis 0 0 1, limit lower=0 upper=1.23 effort=10 velocity=0.8, mimic joint=L_thumb_proximal_pitch_joint multiplier=0.974 offset=0
- added joint L_thumb_proximal_pitch_joint: type revolute, parent L_thumb_proximal_base_link, child L_thumb_proximal_link, origin xyz=0.02175 0 0 rpy=-1.5707 0 0, axis 0 0 1, limit lower=0 upper=1.22 effort=10 velocity=0.8
- added joint L_thumb_proximal_yaw_joint: type revolute, parent L_hand_base_link, child L_thumb_proximal_base_link, origin xyz=0.022 -0.015498 -0.025093 rpy=0 -1.221E-05 0, axis 0 0 1, limit lower=-1.74 upper=0 effort=10 velocity=0.8
- added joint L_thumb_tip_joint: type fixed, parent L_thumb_distal_link, child L_thumb_tip_link, origin xyz=0.031 -0.001 0 rpy=0 0 0
