Commit message: 🎨 modularize configs and updat inspire urdf

File: assets/gr1/urdf/inspire_left_hand.urdf (robot description, URDF)
Before this commit: robot inspire_left_hand, 18 links, 17 joints
Links:
- link L_hand_base_link: geometry collision mesh filename=../meshes/inspire_hand/base_link_l.STL; visual mesh filename=../meshes/inspire_hand/base_link_l.STL
- link L_index_intermediate: geometry collision mesh filename=../meshes/inspire_hand/Link16_l.STL; visual mesh filename=../meshes/inspire_hand/Link16_l.STL
- link L_index_proximal: geometry collision mesh filename=../meshes/inspire_hand/Link15_l.STL; visual mesh filename=../meshes/inspire_hand/Link15_l.STL
- link L_middle_intermediate: geometry collision mesh filename=../meshes/inspire_hand/Link18_l.STL; visual mesh filename=../meshes/inspire_hand/Link18_l.STL
- link L_middle_proximal: geometry collision mesh filename=../meshes/inspire_hand/Link17_l.STL; visual mesh filename=../meshes/inspire_hand/Link17_l.STL
- link L_pinky_intermediate: geometry collision mesh filename=../meshes/inspire_hand/Link22_l.STL; visual mesh filename=../meshes/inspire_hand/Link22_l.STL
- link L_pinky_proximal: geometry collision mesh filename=../meshes/inspire_hand/Link21_l.STL; visual mesh filename=../meshes/inspire_hand/Link21_l.STL
- link L_ring_intermediate: geometry collision mesh filename=../meshes/inspire_hand/Link20_l.STL; visual mesh filename=../meshes/inspire_hand/Link20_l.STL
- link L_ring_proximal: geometry collision mesh filename=../meshes/inspire_hand/Link19_l.STL; visual mesh filename=../meshes/inspire_hand/Link19_l.STL
- link L_thumb_distal: geometry collision mesh filename=../meshes/inspire_hand/Link14_l.STL; visual mesh filename=../meshes/inspire_hand/Link14_l.STL
- link L_thumb_intermediate: geometry collision mesh filename=../meshes/inspire_hand/Link13_l.STL; visual mesh filename=../meshes/inspire_hand/Link13_l.STL
- link L_thumb_proximal: geometry collision mesh filename=../meshes/inspire_hand/Link12_l.STL; visual mesh filename=../meshes/inspire_hand/Link12_l.STL
- link L_thumb_proximal_base: geometry collision mesh filename=../meshes/inspire_hand/Link11_l.STL; visual mesh filename=../meshes/inspire_hand/Link11_l.STL
Joints:
- joint L_index_proximal_joint: origin xyz=0.032268 0.00028533 -0.13653 rpy=1.5708 -0.034907 1.5708 -> xyz=0.00028533 -0.13653 0.032268 rpy=-0.034907 0 0
- joint L_middle_proximal_joint: origin xyz=0.01295 0.00028533 -0.1371 rpy=1.5708 0 1.5708 -> xyz=0.00028533 -0.1371 0.01295 rpy=0 0 0
- joint L_pinky_proximal_joint: origin xyz=-0.025488 0.00028533 -0.13571 rpy=1.5708 0.10472 1.5708 -> xyz=0.00028533 -0.13571 -0.025488 rpy=0.10472 0 0
- joint L_ring_proximal_joint: origin xyz=-0.0062872 0.00028533 -0.13691 rpy=1.5708 0.05236 1.5708 -> xyz=0.00028533 -0.13691 -0.0062872 rpy=0.05236 0 0
- joint L_thumb_proximal_pitch_joint: limit lower=-0.1 upper=0.6 effort=1 velocity=0.5 -> lower=0.0 upper=0.5 effort=1 velocity=0.5
- joint L_thumb_proximal_yaw_joint: origin xyz=0.02045 -0.01696 -0.0691 rpy=3.14 0 0 -> xyz=-0.01696 -0.0691 0.02045 rpy=1.5708 -1.5708 0

File: assets/gr1/urdf/inspire_right_hand.urdf (robot description, URDF)
Before this commit: robot inspire_right_hand, 18 links, 17 joints
Links:
- link R_hand_base_link: geometry collision mesh filename=../meshes/inspire_hand/base_link_r.STL; visual mesh filename=../meshes/inspire_hand/base_link_r.STL
- link R_index_intermediate: geometry collision mesh filename=../meshes/inspire_hand/Link16_r.STL; visual mesh filename=../meshes/inspire_hand/Link16_r.STL
- link R_index_proximal: geometry collision mesh filename=../meshes/inspire_hand/Link15_r.STL; visual mesh filename=../meshes/inspire_hand/Link15_r.STL
- link R_middle_intermediate: geometry collision mesh filename=../meshes/inspire_hand/Link18_r.STL; visual mesh filename=../meshes/inspire_hand/Link18_r.STL
- link R_middle_proximal: geometry collision mesh filename=../meshes/inspire_hand/Link17_r.STL; visual mesh filename=../meshes/inspire_hand/Link17_r.STL
- link R_pinky_intermediate: geometry collision mesh filename=../meshes/inspire_hand/Link22_r.STL; visual mesh filename=../meshes/inspire_hand/Link22_r.STL
- link R_pinky_proximal: geometry collision mesh filename=../meshes/inspire_hand/Link21_r.STL; visual mesh filename=../meshes/inspire_hand/Link21_r.STL
- link R_ring_intermediate: geometry collision mesh filename=../meshes/inspire_hand/Link20_r.STL; visual mesh filename=../meshes/inspire_hand/Link20_r.STL
- link R_ring_proximal: geometry collision mesh filename=../meshes/inspire_hand/Link19_r.STL; visual mesh filename=../meshes/inspire_hand/Link19_r.STL
- link R_thumb_distal: geometry collision mesh filename=../meshes/inspire_hand/Link14_r.STL; visual mesh filename=../meshes/inspire_hand/Link14_r.STL
- link R_thumb_intermediate: geometry collision mesh filename=../meshes/inspire_hand/Link13_r.STL; visual mesh filename=../meshes/inspire_hand/Link13_r.STL
- link R_thumb_proximal: geometry collision mesh filename=../meshes/inspire_hand/Link12_r.STL; visual mesh filename=../meshes/inspire_hand/Link12_r.STL
- link R_thumb_proximal_base: geometry collision mesh filename=../meshes/inspire_hand/Link11_r.STL; visual mesh filename=../meshes/inspire_hand/Link11_r.STL
Joints:
- joint R_index_proximal_joint: origin xyz=0.032268 0.00028533 -0.13653 rpy=-1.5359 0 -1.5708 -> xyz=0.00028533 -0.13653 -0.032268 rpy=-3.1067 0 0
- joint R_middle_proximal_joint: origin xyz=0.01295 0.00028533 -0.1371 rpy=-1.5708 0 -1.5708 -> xyz=0.00028533 -0.1371 -0.01295 rpy=-3.1416 0 0
- joint R_pinky_proximal_joint: origin xyz=-0.025488 0.00028533 -0.13571 rpy=-1.6739 0 -1.5708 -> xyz=0.00028533 -0.13571 0.025488 rpy=3.0369 0 0
- joint R_ring_proximal_joint: origin xyz=-0.0062872 0.00028533 -0.13691 rpy=-1.6232 0 -1.5708 -> xyz=0.00028533 -0.13691 0.0062872 rpy=3.0892 0 0
- joint R_thumb_proximal_pitch_joint: limit lower=-0.1 upper=0.6 effort=1 velocity=0.5 -> lower=0.0 upper=0.5 effort=1 velocity=0.5
- joint R_thumb_proximal_yaw_joint: origin xyz=0.02045 0.01696 -0.0691 rpy=0 3.1416 0 -> xyz=-0.01696 -0.0691 -0.02045 rpy=1.5708 -1.5708 0

Commit message: ✨ unify inspire hand and fourier hand matrix

File: assets/gr1/urdf/inspire_left_hand.urdf (robot description, URDF)
Before this commit: robot inspire_left_hand, 18 links, 17 joints
Links:
- link L_hand_base_link: geometry visual mesh filename=../meshes/inspire_hand/base_link_l.STL
- link L_index_intermediate: geometry visual mesh filename=../meshes/inspire_hand/Link16_l.STL
- link L_index_proximal: geometry visual mesh filename=../meshes/inspire_hand/Link15_l.STL
- link L_middle_intermediate: geometry visual mesh filename=../meshes/inspire_hand/Link18_l.STL
- link L_middle_proximal: geometry visual mesh filename=../meshes/inspire_hand/Link17_l.STL
- link L_pinky_intermediate: geometry visual mesh filename=../meshes/inspire_hand/Link22_l.STL
- link L_pinky_proximal: geometry visual mesh filename=../meshes/inspire_hand/Link21_l.STL
- link L_ring_intermediate: geometry visual mesh filename=../meshes/inspire_hand/Link20_l.STL
- link L_ring_proximal: geometry visual mesh filename=../meshes/inspire_hand/Link19_l.STL
- link L_thumb_distal: geometry visual mesh filename=../meshes/inspire_hand/Link14_l.STL
- link L_thumb_intermediate: geometry visual mesh filename=../meshes/inspire_hand/Link13_l.STL
- link L_thumb_proximal: geometry visual mesh filename=../meshes/inspire_hand/Link12_l.STL
- link L_thumb_proximal_base: geometry visual mesh filename=../meshes/inspire_hand/Link11_l.STL
Joints:
- joint L_index_proximal_joint: origin xyz=0.00028533 -0.13653 0.032268 rpy=-0.034907 0 0 -> xyz=0.032268 0.00028533 -0.13653 rpy=1.5708 -0.034907 1.5708
- joint L_middle_proximal_joint: origin xyz=0.00028533 -0.1371 0.01295 rpy=0 0 0 -> xyz=0.01295 0.00028533 -0.1371 rpy=1.5708 0 1.5708
- joint L_pinky_proximal_joint: origin xyz=0.00028533 -0.13571 -0.025488 rpy=0.10472 0 0 -> xyz=-0.025488 0.00028533 -0.13571 rpy=1.5708 0.10472 1.5708
- joint L_ring_proximal_joint: origin xyz=0.00028533 -0.13691 -0.0062872 rpy=0.05236 0 0 -> xyz=-0.0062872 0.00028533 -0.13691 rpy=1.5708 0.05236 1.5708
- joint L_thumb_proximal_pitch_joint: limit lower=0.0 upper=0.5 effort=1 velocity=0.5 -> lower=-0.1 upper=0.6 effort=1 velocity=0.5
- joint L_thumb_proximal_yaw_joint: origin xyz=-0.01696 -0.0691 0.02045 rpy=1.5708 -1.5708 0 -> xyz=0.02045 -0.01696 -0.0691 rpy=3.14 0 0

File: assets/gr1/urdf/inspire_right_hand.urdf (robot description, URDF)
Before this commit: robot inspire_right_hand, 18 links, 17 joints
Links:
- link R_hand_base_link: geometry visual mesh filename=../meshes/inspire_hand/base_link_r.STL
- link R_index_intermediate: geometry visual mesh filename=../meshes/inspire_hand/Link16_r.STL
- link R_index_proximal: geometry visual mesh filename=../meshes/inspire_hand/Link15_r.STL
- link R_middle_intermediate: geometry visual mesh filename=../meshes/inspire_hand/Link18_r.STL
- link R_middle_proximal: geometry visual mesh filename=../meshes/inspire_hand/Link17_r.STL
- link R_pinky_intermediate: geometry visual mesh filename=../meshes/inspire_hand/Link22_r.STL
- link R_pinky_proximal: geometry visual mesh filename=../meshes/inspire_hand/Link21_r.STL
- link R_ring_intermediate: geometry visual mesh filename=../meshes/inspire_hand/Link20_r.STL
- link R_ring_proximal: geometry visual mesh filename=../meshes/inspire_hand/Link19_r.STL
- link R_thumb_distal: geometry visual mesh filename=../meshes/inspire_hand/Link14_r.STL
- link R_thumb_intermediate: geometry visual mesh filename=../meshes/inspire_hand/Link13_r.STL
- link R_thumb_proximal: geometry visual mesh filename=../meshes/inspire_hand/Link12_r.STL
- link R_thumb_proximal_base: geometry visual mesh filename=../meshes/inspire_hand/Link11_r.STL
Joints:
- joint R_index_proximal_joint: origin xyz=0.00028533 -0.13653 -0.032268 rpy=-3.1067 0 0 -> xyz=0.032268 0.00028533 -0.13653 rpy=-1.5359 0 -1.5708
- joint R_middle_proximal_joint: origin xyz=0.00028533 -0.1371 -0.01295 rpy=-3.1416 0 0 -> xyz=0.01295 0.00028533 -0.1371 rpy=-1.5708 0 -1.5708
- joint R_pinky_proximal_joint: origin xyz=0.00028533 -0.13571 0.025488 rpy=3.0369 0 0 -> xyz=-0.025488 0.00028533 -0.13571 rpy=-1.6739 0 -1.5708
- joint R_ring_proximal_joint: origin xyz=0.00028533 -0.13691 0.0062872 rpy=3.0892 0 0 -> xyz=-0.0062872 0.00028533 -0.13691 rpy=-1.6232 0 -1.5708
- joint R_thumb_proximal_pitch_joint: limit lower=0.0 upper=0.5 effort=1 velocity=0.5 -> lower=-0.1 upper=0.6 effort=1 velocity=0.5
- joint R_thumb_proximal_yaw_joint: origin xyz=-0.01696 -0.0691 -0.02045 rpy=1.5708 -1.5708 0 -> xyz=0.02045 0.01696 -0.0691 rpy=0 3.1416 0
