Commit message: 🍱 update urdf
Signed-off-by: Yuxiang Gao <yuxiang.gao@fftai.com>

File: assets/urdf/qinglong_fourier_hand_6dof.urdf (robot description, URDF)
Before this commit: robot openloong_fourier_hand_6dof, 70 links, 69 joints
Links:
- link L_hand_camera_frame_link: geometry collision mesh filename=../meshes/qinglong/left_camera_frame_link.STL; visual mesh filename=../meshes/qinglong/left_camera_frame_link.STL
- link R_hand_camera_frame_link: geometry collision mesh filename=../meshes/qinglong/right_camera_frame_link.STL; visual mesh filename=../meshes/qinglong/right_camera_frame_link.STL
- link left_end_effector_link: geometry collision mesh filename=../meshes/qinglong/left_end_effector_link.STL; visual mesh filename=../meshes/qinglong/left_end_effector_link.STL
- link right_end_effector_link: mass 0.018 -> 0.018343; geometry collision mesh filename=../meshes/qinglong/right_end_effecotr_link.STL; visual mesh filename=../meshes/qinglong/right_end_effecotr_link.STL
Joints:
- joint L_hand_base_joint: origin xyz=0.028 0.028 0.009 rpy=0 0 0 -> xyz=0 0 0.0045 rpy=0 0 0
- joint L_hand_camera_frame_joint: origin xyz=-0.0282 -0.027 -0.011 rpy=0 0 0 -> xyz=0 0 -0.004 rpy=0 0 0
- joint R_hand_base_joint: origin xyz=0.028 0.028 0.0088 rpy=0 0 0 -> xyz=0 0 0.0045 rpy=0 0 0
- joint R_hand_camera_frame_joint: origin xyz=-0.0282 -0.027 -0.011 rpy=0 0 0 -> xyz=0 0 -0.003 rpy=0 0 0
- joint left_end_effector_joint: origin xyz=-0.0282 0.082 -0.06 rpy=1.57 0 0 -> xyz=0.0 0.0760 -0.031 rpy=1.57 0 0
- joint right_end_effector_joint: origin xyz=-0.0282 -0.082 -0.00345 rpy=-1.57 0 0 -> xyz=0.0 -0.0760 -0.031 rpy=-1.57 0 0
