Commit message: 🐛 fix end_effector_link in gr2 urdf
Signed-off-by: Yuxiang Gao <yuxiang.gao@fftai.com>

File: assets/urdf/GR2T2_fourier_hand_12dof.urdf (robot description, URDF)
Before this commit: robot GR2T2_fourier_hand_12dof, 71 links, 70 joints
Joints:
- joint L_hand_base_joint: origin xyz=0 0 -0.043 rpy=0 0 0 -> xyz=0 0 0 rpy=0 0 0
- joint R_hand_base_joint: origin xyz=0 0 -0.043 rpy=0 0 0 -> xyz=0 0 0 rpy=0 0 0
- joint left_end_effector_joint: origin xyz=0 0 0 rpy=0 0 0 -> xyz=0 0 -0.043 rpy=0 0 0
- joint right_end_effector_joint: origin xyz=0 0 0 rpy=0 0 0 -> xyz=0 0 -0.043 rpy=0 0 0

File: assets/urdf/GR2T2_fourier_hand_6dof.urdf (robot description, URDF)
Before this commit: robot GR2T2_fourier_hand_6dof, 69 links, 68 joints
Joints:
- joint L_hand_base_joint: origin xyz=0 0 -0.043 rpy=0 0 0 -> xyz=0 0 0 rpy=0 0 0
- joint R_hand_base_joint: origin xyz=0 0 -0.043 rpy=-6.83500415935726E-05 1.22100046026127E-05 0 -> xyz=0 0 0 rpy=-6.83500415935726E-05 1.22100046026127E-05 0
- joint left_end_effector_joint: origin xyz=0 0 0 rpy=0 0 0 -> xyz=0 0 -0.043 rpy=0 0 0
- joint right_end_effector_joint: origin xyz=0 0 0 rpy=0 0 0 -> xyz=0 0 -0.043 rpy=0 0 0
