Commit message: server_config and hand config with metacarpal's direction

File: server_config/fourier_hardware/gr2t2/robot.urdf (robot description, URDF)
Before this commit: robot GR2T2, 35 links, 34 joints
Links:
- link base_link: geometry collision sphere radius=0.05; collision sphere radius=0.05
- link camera_link: geometry visual mesh filename=../../../assets/meshes/gr2t2/camera_link.STL
- link head_pitch_link: geometry collision sphere radius=0.08; visual mesh filename=../../../assets/meshes/gr2t2/head_pitch_link.STL
- link head_yaw_link: geometry visual mesh filename=../../../assets/meshes/gr2t2/head_yaw_link.STL
- link imu_link: geometry visual mesh filename=../../../assets/meshes/gr2t2/imu_link.STL
- link left_end_effector_link: geometry collision sphere radius=0.035; visual mesh filename=../../../assets/meshes/gr2t2/left_end_effector_link.STL
- link left_foot_pitch_link: geometry collision mesh filename=../../../assets/meshes/gr2t2/left_foot_pitch_link.STL; visual mesh filename=../../../assets/meshes/gr2t2/left_foot_pitch_link.STL
- link left_foot_roll_link: geometry visual mesh filename=../../../assets/meshes/gr2t2/left_foot_roll_link.STL
- link left_hand_pitch_link: geometry visual mesh filename=../../../assets/meshes/gr2t2/left_hand_pitch_link.STL
- link left_hand_roll_link: geometry visual mesh filename=../../../assets/meshes/gr2t2/left_hand_roll_link.STL
- link left_hand_yaw_link: geometry collision cylinder length=0.17 radius=0.035; visual mesh filename=../../../assets/meshes/gr2t2/left_hand_yaw_link.STL
- link left_lower_arm_pitch_link: geometry visual mesh filename=../../../assets/meshes/gr2t2/left_lower_arm_pitch_link.STL
- link left_shank_pitch_link: geometry collision cylinder length=0.2 radius=0.05; visual mesh filename=../../../assets/meshes/gr2t2/left_shank_pitch_link.STL
- link left_thigh_pitch_link: geometry visual mesh filename=../../../assets/meshes/gr2t2/left_thigh_pitch_link.STL
- link left_thigh_roll_link: geometry visual mesh filename=../../../assets/meshes/gr2t2/left_thigh_roll_link.STL
- link left_thigh_yaw_link: geometry collision cylinder length=0.25 radius=0.05; visual mesh filename=../../../assets/meshes/gr2t2/left_thigh_yaw_link.STL
- link left_upper_arm_pitch_link: geometry visual mesh filename=../../../assets/meshes/gr2t2/left_upper_arm_pitch_link.STL
- link left_upper_arm_roll_link: geometry visual mesh filename=../../../assets/meshes/gr2t2/left_upper_arm_roll_link.STL
- link left_upper_arm_yaw_link: geometry collision cylinder length=0.11 radius=0.03; visual mesh filename=../../../assets/meshes/gr2t2/left_upper_arm_yaw_link.STL
- link right_end_effector_link: geometry collision sphere radius=0.035; visual mesh filename=../../../assets/meshes/gr2t2/right_end_effector_link.STL
- link right_foot_pitch_link: geometry collision mesh filename=../../../assets/meshes/gr2t2/right_foot_pitch_link.STL; visual mesh filename=../../../assets/meshes/gr2t2/right_foot_pitch_link.STL
- link right_foot_roll_link: geometry visual mesh filename=../../../assets/meshes/gr2t2/right_foot_roll_link.STL
- link right_hand_pitch_link: geometry visual mesh filename=../../../assets/meshes/gr2t2/right_hand_pitch_link.STL
- link right_hand_roll_link: geometry visual mesh filename=../../../assets/meshes/gr2t2/right_hand_roll_link.STL
- link right_hand_yaw_link: geometry collision cylinder length=0.17 radius=0.035; visual mesh filename=../../../assets/meshes/gr2t2/right_hand_yaw_link.STL
- link right_lower_arm_pitch_link: geometry visual mesh filename=../../../assets/meshes/gr2t2/right_lower_arm_pitch_link.STL
- link right_shank_pitch_link: geometry collision cylinder length=0.2 radius=0.05; visual mesh filename=../../../assets/meshes/gr2t2/right_shank_pitch_link.STL
- link right_thigh_pitch_link: geometry visual mesh filename=../../../assets/meshes/gr2t2/right_thigh_pitch_link.STL
- link right_thigh_roll_link: geometry visual mesh filename=../../../assets/meshes/gr2t2/right_thigh_roll_link.STL
- link right_thigh_yaw_link: geometry collision cylinder length=0.25 radius=0.05; visual mesh filename=../../../assets/meshes/gr2t2/right_thigh_yaw_link.STL
- link right_upper_arm_pitch_link: geometry visual mesh filename=../../../assets/meshes/gr2t2/right_upper_arm_pitch_link.STL
- link right_upper_arm_roll_link: geometry visual mesh filename=../../../assets/meshes/gr2t2/right_upper_arm_roll_link.STL
- link right_upper_arm_yaw_link: geometry collision cylinder length=0.11 radius=0.03; visual mesh filename=../../../assets/meshes/gr2t2/right_upper_arm_yaw_link.STL
- link torso_link: geometry collision cylinder length=0.25 radius=0.1; visual mesh filename=../../../assets/meshes/gr2t2/torso_link.STL
- link waist_yaw_link: geometry visual mesh filename=../../../assets/meshes/gr2t2/waist_yaw_link.STL
